Commit message: tf created

File: fixi_description/urdf/fixi.urdf.xacro (robot description, xacro)
@@ -36,4 +36,33 @@
         izz="${mass * radius * radius / 2.0}"/>
     </inertial>
+  </xacro:macro>
+  <xacro:macro name="ultrasonic_sensor" params="name x y z yaw">
+    <link name="${name}_ultrasonic_link">
+      <visual>
+        <origin xyz="0 0 0" rpy="0 0 0"/>
+        <geometry>
+          <box size="0.035 0.055 0.025"/>
+        </geometry>
+        <material name="fixi_blue"/>
+      </visual>
+      <collision>
+        <origin xyz="0 0 0" rpy="0 0 0"/>
+        <geometry>
+          <box size="0.035 0.055 0.025"/>
+        </geometry>
+      </collision>
+      <xacro:box_inertial mass="0.05" x="0.035" y="0.055" z="0.025"/>
+    </link>
+    <joint name="${name}_ultrasonic_joint" type="fixed">
+      <parent link="base_link"/>
+      <child link="${name}_ultrasonic_link"/>
+      <origin xyz="${x} ${y} ${z}" rpy="0 0 ${yaw}"/>
+    </joint>
+    <link name="${name}_ultrasonic_frame"/>
+    <joint name="${name}_ultrasonic_frame_joint" type="fixed">
+      <parent link="${name}_ultrasonic_link"/>
+      <child link="${name}_ultrasonic_frame"/>
+      <origin xyz="0.025 0 0" rpy="0 0 0"/>
+    </joint>
   </xacro:macro>
   <material name="fixi_teal">
@@ -191,4 +220,28 @@
     <origin xyz="0.025 0 0" rpy="-1.5708 0 -1.5708"/>
   </joint>
+  <xacro:ultrasonic_sensor
+    name="front"
+    x="${base_length / 2.0 + 0.015}"
+    y="0"
+    z="0.02"
+    yaw="0"/>
+  <xacro:ultrasonic_sensor
+    name="left"
+    x="0.02"
+    y="${base_width / 2.0 + 0.015}"
+    z="0.02"
+    yaw="1.5708"/>
+  <xacro:ultrasonic_sensor
+    name="right"
+    x="0.02"
+    y="${-base_width / 2.0 - 0.015}"
+    z="0.02"
+    yaw="-1.5708"/>
+  <xacro:ultrasonic_sensor
+    name="rear"
+    x="${-base_length / 2.0 - 0.015}"
+    y="0"
+    z="0.02"
+    yaw="3.1416"/>
   <link name="storage_bin_link">
     <visual>
@@ -391,4 +444,11 @@
     <axis xyz="0 -1 0"/>
     <limit lower="0.0" upper="0.035" effort="2.0" velocity="0.05"/>
+    <mimic joint="left_gripper_finger_joint" multiplier="1.0" offset="0.0"/>
+  </joint>
+  <link name="gripper_tcp"/>
+  <joint name="gripper_tcp_joint" type="fixed">
+    <parent link="gripper_base_link"/>
+    <child link="gripper_tcp"/>
+    <origin xyz="0.14 0 0" rpy="0 0 0"/>
   </joint>
 </robot>
