Commit message: error fix in teleop

File: fixi_description/urdf/fixi.gazebo.xacro (robot description, xacro)
@@ -8,29 +8,40 @@
       <plugin>gz_ros2_control/GazeboSimSystem</plugin>
     </hardware>
-    <joint name="left_wheel_joint">
-      <command_interface name="velocity">
-        <param name="min">-10.0</param>
-        <param name="max">10.0</param>
-      </command_interface>
+    <joint name="arm_joint_1_yaw">
       <state_interface name="position"/>
-      <state_interface name="velocity"/>
     </joint>
-    <joint name="right_wheel_joint">
-      <command_interface name="velocity">
-        <param name="min">-10.0</param>
-        <param name="max">10.0</param>
-      </command_interface>
+    <joint name="arm_joint_2_shoulder">
       <state_interface name="position"/>
-      <state_interface name="velocity"/>
+    </joint>
+    <joint name="arm_joint_3_elbow">
+      <state_interface name="position"/>
+    </joint>
+    <joint name="arm_joint_4_wrist">
+      <state_interface name="position"/>
+    </joint>
+    <joint name="left_gripper_finger_joint">
+      <state_interface name="position"/>
+    </joint>
+    <joint name="right_gripper_finger_joint">
+      <state_interface name="position"/>
     </joint>
   </ros2_control>
   <gazebo>
-    <plugin filename="gz_ros2_control-system" name="gz_ros2_control::GazeboSimSystem">
+    <plugin filename="gz_ros2_control-system" name="gz_ros2_control::GazeboSimROS2ControlPlugin">
       <parameters>$(find fixi_gazebo)/config/ros2_controllers.yaml</parameters>
     </plugin>
-    <plugin
-      filename="gz-sim-sensors-system"
-      name="gz::sim::systems::Sensors">
-      <render_engine>ogre2</render_engine>
+    <plugin filename="gz-sim-diff-drive-system" name="gz::sim::systems::DiffDrive">
+      <left_joint>front_left_wheel_joint</left_joint>
+      <right_joint>front_right_wheel_joint</right_joint>
+      <wheel_separation>0.485</wheel_separation>
+      <wheel_radius>0.075</wheel_radius>
+      <topic>/cmd_vel</topic>
+    </plugin>
+    <plugin filename="gz-sim-diff-drive-system" name="gz::sim::systems::DiffDrive">
+      <left_joint>rear_left_wheel_joint</left_joint>
+      <right_joint>rear_right_wheel_joint</right_joint>
+      <wheel_separation>0.485</wheel_separation>
+      <wheel_radius>0.075</wheel_radius>
+      <topic>/cmd_vel</topic>
     </plugin>
   </gazebo>
@@ -39,22 +50,20 @@
   <!-- ============================================ -->
   <gazebo reference="base_link">
-    <material>Gazebo/Blue</material>
   </gazebo>
-  <gazebo reference="left_wheel_link">
-    <material>Gazebo/DarkGrey</material>
+  <gazebo reference="front_left_wheel_link">
     <mu1>1.0</mu1>
     <mu2>1.0</mu2>
   </gazebo>
-  <gazebo reference="right_wheel_link">
-    <material>Gazebo/DarkGrey</material>
+  <gazebo reference="front_right_wheel_link">
     <mu1>1.0</mu1>
     <mu2>1.0</mu2>
   </gazebo>
-  <gazebo reference="caster_wheel_link">
-    <material>Gazebo/Grey</material>
-    <mu1>0.001</mu1>
-    <mu2>0.001</mu2>
-    <kp>1000000.0</kp>
-    <kd>100.0</kd>
+  <gazebo reference="rear_left_wheel_link">
+    <mu1>1.0</mu1>
+    <mu2>1.0</mu2>
+  </gazebo>
+  <gazebo reference="rear_right_wheel_link">
+    <mu1>1.0</mu1>
+    <mu2>1.0</mu2>
   </gazebo>
   <!-- ============================================ -->
@@ -67,4 +76,5 @@
       <update_rate>30.0</update_rate>
       <topic>camera/image_raw</topic>
+      <gz_frame_id>camera_optical_frame</gz_frame_id>
       <camera name="head">
         <horizontal_fov>1.3962634</horizontal_fov>

File: fixi_description/urdf/fixi.urdf.xacro (robot description, xacro)
@@ -6,7 +6,7 @@
   <xacro:property name="wheel_radius" value="0.075"/>
   <xacro:property name="wheel_width" value="0.045"/>
-  <xacro:property name="wheel_y" value="${base_width / 2.0 + wheel_width / 2.0}"/>
+  <xacro:property name="wheel_y" value="${base_width / 2.0 + wheel_width / 2.0 + 0.01}"/>
   <xacro:property name="wheel_x" value="-0.04"/>
-  <xacro:property name="wheel_z" value="${wheel_radius}"/>
+  <xacro:property name="wheel_z" value="0.05"/>
   <xacro:property name="caster_radius" value="0.035"/>
   <xacro:property name="arm_base_z" value="${base_height + 0.035}"/>
@@ -40,9 +40,9 @@
     <link name="${name}_ultrasonic_link">
       <visual>
+      <material name="mat_1"><color rgba="0.401 0.5 0.5 1.0"/></material>
         <origin xyz="0 0 0" rpy="0 0 0"/>
         <geometry>
           <box size="0.035 0.055 0.025"/>
         </geometry>
-        <material name="fixi_blue"/>
       </visual>
       <collision>
@@ -66,19 +66,4 @@
     </joint>
   </xacro:macro>
-  <material name="fixi_teal">
-    <color rgba="0.0 0.55 0.50 1.0"/>
-  </material>
-  <material name="fixi_dark">
-    <color rgba="0.08 0.09 0.10 1.0"/>
-  </material>
-  <material name="fixi_gray">
-    <color rgba="0.45 0.48 0.50 1.0"/>
-  </material>
-  <material name="fixi_blue">
-    <color rgba="0.05 0.25 0.80 1.0"/>
-  </material>
-  <material name="fixi_clear">
-    <color rgba="0.30 0.80 1.00 0.45"/>
-  </material>
   <link name="base_footprint"/>
   <joint name="base_footprint_to_base_link" type="fixed">
@@ -89,9 +74,9 @@
   <link name="base_link">
     <visual>
+      <material name="mat_2"><color rgba="0.402 0.5 0.5 1.0"/></material>
       <origin xyz="0 0 0" rpy="0 0 0"/>
       <geometry>
         <box size="${base_length} ${base_width} ${base_height}"/>
       </geometry>
-      <material name="fixi_teal"/>
     </visual>
     <collision>
@@ -103,80 +88,41 @@
     <xacro:box_inertial mass="8.0" x="${base_length}" y="${base_width}" z="${base_height}"/>
   </link>
-  <link name="left_wheel_link">
-    <visual>
-      <origin xyz="0 0 0" rpy="1.5708 0 0"/>
-      <geometry>
-        <cylinder radius="${wheel_radius}" length="${wheel_width}"/>
-      </geometry>
-      <material name="fixi_dark"/>
-    </visual>
-    <collision>
-      <origin xyz="0 0 0" rpy="1.5708 0 0"/>
-      <geometry>
-        <cylinder radius="${wheel_radius}" length="${wheel_width}"/>
-      </geometry>
-    </collision>
-    <xacro:cylinder_inertial mass="0.6" radius="${wheel_radius}" length="${wheel_width}"/>
-  </link>
-  <joint name="left_wheel_joint" type="continuous">
-    <parent link="base_link"/>
-    <child link="left_wheel_link"/>
-    <origin xyz="${wheel_x} ${wheel_y} ${-base_height / 2.0 + wheel_z}" rpy="0 0 0"/>
-    <axis xyz="0 1 0"/>
-  </joint>
-  <link name="right_wheel_link">
-    <visual>
-      <origin xyz="0 0 0" rpy="1.5708 0 0"/>
-      <geometry>
-        <cylinder radius="${wheel_radius}" length="${wheel_width}"/>
-      </geometry>
-      <material name="fixi_dark"/>
-    </visual>
-    <collision>
-      <origin xyz="0 0 0" rpy="1.5708 0 0"/>
-      <geometry>
-        <cylinder radius="${wheel_radius}" length="${wheel_width}"/>
-      </geometry>
-    </collision>
-    <xacro:cylinder_inertial mass="0.6" radius="${wheel_radius}" length="${wheel_width}"/>
-  </link>
-  <joint name="right_wheel_joint" type="continuous">
-    <parent link="base_link"/>
-    <child link="right_wheel_link"/>
-    <origin xyz="${wheel_x} ${-wheel_y} ${-base_height / 2.0 + wheel_z}" rpy="0 0 0"/>
-    <axis xyz="0 1 0"/>
-  </joint>
-  <link name="caster_wheel_link">
-    <visual>
-      <origin xyz="0 0 0" rpy="0 0 0"/>
-      <geometry>
-        <sphere radius="${caster_radius}"/>
-      </geometry>
-      <material name="fixi_gray"/>
-    </visual>
-    <collision>
-      <origin xyz="0 0 0" rpy="0 0 0"/>
-      <geometry>
-        <sphere radius="${caster_radius}"/>
-      </geometry>
-    </collision>
-    <inertial>
-      <mass value="0.2"/>
-      <origin xyz="0 0 0" rpy="0 0 0"/>
-      <inertia ixx="0.0001" ixy="0" ixz="0" iyy="0.0001" iyz="0" izz="0.0001"/>
-    </inertial>
-  </link>
-  <joint name="caster_wheel_joint" type="fixed">
-    <parent link="base_link"/>
-    <child link="caster_wheel_link"/>
-    <origin xyz="0.22 0 ${-base_height / 2.0 + caster_radius}" rpy="0 0 0"/>
-  </joint>
+  <xacro:property name="wheel_x_offset" value="0.18"/>
+  <xacro:macro name="drive_wheel" params="prefix x_reflect y_reflect mat_id">
+    <link name="${prefix}_wheel_link">
+      <visual>
+        <material name="mat_${mat_id}"><color rgba="0.4 0.5 0.5 1.0"/></material>
+        <origin xyz="0 0 0" rpy="1.5708 0 0"/>
+        <geometry>
+          <cylinder radius="${wheel_radius}" length="${wheel_width}"/>
+        </geometry>
+      </visual>
+      <collision>
+        <origin xyz="0 0 0" rpy="1.5708 0 0"/>
+        <geometry>
+          <cylinder radius="${wheel_radius}" length="${wheel_width}"/>
+        </geometry>
+      </collision>
+      <xacro:cylinder_inertial mass="0.6" radius="${wheel_radius}" length="${wheel_width}"/>
+    </link>
+    <joint name="${prefix}_wheel_joint" type="continuous">
+      <parent link="base_link"/>
+      <child link="${prefix}_wheel_link"/>
+      <origin xyz="${wheel_x_offset * x_reflect} ${wheel_y * y_reflect} ${-base_height / 2.0 + wheel_z}" rpy="0 0 0"/>
+      <axis xyz="0 1 0"/>
+      <limit effort="100.0" velocity="20.0"/>
+    </joint>
+  </xacro:macro>
+  <xacro:drive_wheel prefix="front_left" x_reflect="1" y_reflect="1" mat_id="101"/>
+  <xacro:drive_wheel prefix="front_right" x_reflect="1" y_reflect="-1" mat_id="102"/>
+  <xacro:drive_wheel prefix="rear_left" x_reflect="-1" y_reflect="1" mat_id="103"/>
+  <xacro:drive_wheel prefix="rear_right" x_reflect="-1" y_reflect="-1" mat_id="104"/>
   <link name="camera_mount_link">
     <visual>
+      <material name="mat_6"><color rgba="0.406 0.5 0.5 1.0"/></material>
       <origin xyz="0 0 0" rpy="0 0 0"/>
       <geometry>
         <box size="0.10 0.08 0.05"/>
       </geometry>
-      <material name="fixi_dark"/>
     </visual>
     <collision>
@@ -195,9 +141,9 @@
   <link name="camera_link">
     <visual>
+      <material name="mat_7"><color rgba="0.40700000000000003 0.5 0.5 1.0"/></material>
       <origin xyz="0 0 0" rpy="0 0 0"/>
       <geometry>
         <box size="0.045 0.09 0.045"/>
       </geometry>
-      <material name="fixi_blue"/>
     </visual>
     <collision>
@@ -246,9 +192,9 @@
   <link name="storage_bin_link">
     <visual>
+      <material name="mat_8"><color rgba="0.40800000000000003 0.5 0.5 1.0"/></material>
       <origin xyz="0 0 0" rpy="0 0 0"/>
       <geometry>
         <box size="0.22 0.32 0.18"/>
       </geometry>
-      <material name="fixi_clear"/>
     </visual>
     <collision>
@@ -267,9 +213,9 @@
   <link name="arm_base_link">
     <visual>
+      <material name="mat_9"><color rgba="0.40900000000000003 0.5 0.5 1.0"/></material>
       <origin xyz="0 0 0.025" rpy="0 0 0"/>
       <geometry>
         <cylinder radius="0.055" length="0.05"/>
       </geometry>
-      <material name="fixi_gray"/>
     </visual>
     <collision>
@@ -288,9 +234,9 @@
   <link name="arm_shoulder_link">
     <visual>
+      <material name="mat_10"><color rgba="0.41000000000000003 0.5 0.5 1.0"/></material>
       <origin xyz="0 0 0.08" rpy="0 0 0"/>
       <geometry>
         <box size="0.055 0.055 0.16"/>
       </geometry>
-      <material name="fixi_gray"/>
     </visual>
     <collision>
@@ -311,9 +257,9 @@
   <link name="arm_upper_link">
     <visual>
+      <material name="mat_11"><color rgba="0.41100000000000003 0.5 0.5 1.0"/></material>
       <origin xyz="0.10 0 0" rpy="0 1.5708 0"/>
       <geometry>
         <cylinder radius="0.027" length="0.20"/>
       </geometry>
-      <material name="fixi_teal"/>
     </visual>
     <collision>
@@ -334,9 +280,9 @@
   <link name="arm_forearm_link">
     <visual>
+      <material name="mat_12"><color rgba="0.41200000000000003 0.5 0.5 1.0"/></material>
       <origin xyz="0.09 0 0" rpy="0 1.5708 0"/>
       <geometry>
         <cylinder radius="0.024" length="0.18"/>
       </geometry>
-      <material name="fixi_teal"/>
     </visual>
     <collision>
@@ -357,9 +303,9 @@
   <link name="arm_wrist_link">
     <visual>
+      <material name="mat_13"><color rgba="0.41300000000000003 0.5 0.5 1.0"/></material>
       <origin xyz="0.045 0 0" rpy="0 1.5708 0"/>
       <geometry>
         <cylinder radius="0.022" length="0.09"/>
       </geometry>
-      <material name="fixi_gray"/>
     </visual>
     <collision>
@@ -380,9 +326,9 @@
   <link name="gripper_base_link">
     <visual>
+      <material name="mat_14"><color rgba="0.41400000000000003 0.5 0.5 1.0"/></material>
       <origin xyz="0.025 0 0" rpy="0 0 0"/>
       <geometry>
         <box size="0.05 0.08 0.035"/>
       </geometry>
-      <material name="fixi_dark"/>
     </visual>
     <collision>
@@ -401,9 +347,9 @@
   <link name="left_gripper_finger_link">
     <visual>
+      <material name="mat_15"><color rgba="0.41500000000000004 0.5 0.5 1.0"/></material>
       <origin xyz="0.04 0 0" rpy="0 0 0"/>
       <geometry>
         <box size="0.08 0.018 0.025"/>
       </geometry>
-      <material name="fixi_gray"/>
     </visual>
     <collision>
@@ -424,9 +370,9 @@
   <link name="right_gripper_finger_link">
     <visual>
+      <material name="mat_16"><color rgba="0.41600000000000004 0.5 0.5 1.0"/></material>
       <origin xyz="0.04 0 0" rpy="0 0 0"/>
       <geometry>
         <box size="0.08 0.018 0.025"/>
       </geometry>
-      <material name="fixi_gray"/>
     </visual>
     <collision>
